File: Ultramarine-2.kicad_sch (KiCad schematic)
At the start: 51 parts, among them J1 OLED, J2 TRRS, SW1 SW_Push, SW10 SW_Push, SW11 SW_Push, SW12 SW_Push, SW13 SW_Push, SW14 SW_Push, SW15 SW_Push, SW16 SW_Push, SW17 SW_Push, SW18 SW_Push, SW19 SW_Push, SW2 SW_Push, SW20 SW_Push, SW21 SW_Push, SW22 SW_Push, SW23 SW_Push, SW24 SW_Push, SW25 SW_Push, SW26 SW_Push, SW27 SW_Push, SW28 SW_Push, SW29 SW_Push, SW3 SW_Push, SW30 SW_Push, SW31 SW_Push, SW32 SW_Push, SW33 SW_Push, SW34 SW_Push, SW35 SW_Push, SW36 SW_Push, SW4 SW_Push, SW5 SW_Push, SW6 SW_Push, SW7 SW_Push, SW8 SW_Push, SW9 SW_Push

Commit message: add PCB dxf file
Parts:
- removed SW28, SW32: SW_Push, Ultramarine-2:MX-Kailh, symbol Switch:SW_Push
- added C1, C2: C, Capacitor_SMD:C_0603_1608Metric, symbol Device:C
- added D1, D10, D11, D12, D13, D14, D2, D22, D23, D24, D25, D26, D27, D28, D29, D3, D30, D31, D32, D33, D34, D35, D4, D43, D44, D45, D46, D47, D48, D49, D5, D50, D51, D52, D53, D54, D55, D56, D6, D64, D65, D66, D67, D68, D69, D7, D70, D71, D72, D73, D74, D75, D76, D77, D8, D85, D86, D87, D88, D89, D9, D90, D91, D92, D93, D94, D95, D96, D97, D98: SK6812MINI, LED_SMD:LED_SK6812MINI_PLCC4_3.5x3.5mm_P1.75mm, symbol LED:SK6812MINI
- added D100, D101, D102, D103, D104, D105, D16, D17, D18, D19, D20, D21, D36, D37, D38, D39, D40, D41, D42, D57, D58, D59, D60, D61, D62, D63, D78, D79, D80, D81, D82, D83, D84, D99: D, Diode_SMD:D_SOD-123, symbol Device:D
- added J3: Qi Charging unit, symbol Connector:Conn_01x02_Socket
- added J4: LiPo, symbol Connector:Conn_01x02_Socket
- added SW31: Extra, Button_Switch_THT:SW_Tactile_SPST_Angled_PTS645Vx58-2LFS, symbol Switch:SW_Push
- added SW35: RotaryEncoder_Switch, Rotary_Encoder:RotaryEncoder_Alps_EC12E-Switch_Vertical_H20mm, symbol Device:RotaryEncoder_Switch
- added SW37: Power Switch, symbol Switch:SW_Push_SPDT
- added U1: ~, Package_TO_SOT_SMD:SOT-89-5, symbol Ultramarine-2:NJM2884
- JP1: value Jumper_3_Open -> OLED Jumper1
- JP2: value Jumper_3_Open -> OLED Jumper2
- JP3: value Jumper_3_Open -> OLED Jumper3
- JP4: value Jumper_3_Open -> OLED Jumper4
- SW14: value SW_Push -> Command 2; footprint Ultramarine-2:MX-Kailh -> Button_Switch_THT:SW_Tactile_SPST_Angled_PTS645Vx58-2LFS
- SW21: value SW_Push -> Command 3; footprint Ultramarine-2:MX-Kailh -> Button_Switch_THT:SW_Tactile_SPST_Angled_PTS645Vx58-2LFS
- SW36: value SW_Push -> Reset; footprint Ultramarine-2:MX-Kailh -> Button_Switch_THT:SW_Tactile_SPST_Angled_PTS645Vx58-2LFS
- SW7: value SW_Push -> Command 1; footprint Ultramarine-2:MX-Kailh -> Button_Switch_THT:SW_Tactile_SPST_Angled_PTS645Vx58-2LFS
- renumbered D1 to D106, D2 to D107, D3 to D15, SW29 to SW28, SW30 to SW29, SW31 to SW30, SW33 to SW32, SW34 to SW33, SW35 to SW34
Connections:
- net +5V: now also J2.1 (Pin_1), D1.4 (VDD), D10.4 (VDD), D11.4 (VDD), D12.4 (VDD), D13.4 (VDD), D14.4 (VDD), D2.4 (VDD), D22.4 (VDD), D23.4 (VDD), D24.4 (VDD), D25.4 (VDD), D26.4 (VDD), D27.4 (VDD), D28.4 (VDD), D29.4 (VDD), D3.4 (VDD), D30.4 (VDD), D31.4 (VDD), D32.4 (VDD), D33.4 (VDD), D34.4 (VDD), D35.4 (VDD), D4.4 (VDD), D43.4 (VDD), D44.4 (VDD), D45.4 (VDD), D46.4 (VDD), D47.4 (VDD), D48.4 (VDD), D49.4 (VDD), D5.4 (VDD), D50.4 (VDD), D51.4 (VDD), D52.4 (VDD), D53.4 (VDD), D54.4 (VDD), D55.4 (VDD), D56.4 (VDD), D6.4 (VDD), D64.4 (VDD), D65.4 (VDD), D66.4 (VDD), D67.4 (VDD), D68.4 (VDD), D69.4 (VDD), D7.4 (VDD), D70.4 (VDD), D71.4 (VDD), D72.4 (VDD), D73.4 (VDD), D74.4 (VDD), D75.4 (VDD), D76.4 (VDD), D77.4 (VDD), D8.4 (VDD), D85.4 (VDD), D86.4 (VDD), D87.4 (VDD), D88.4 (VDD), D89.4 (VDD), D9.4 (VDD), D90.4 (VDD), D91.4 (VDD), D92.4 (VDD), D93.4 (VDD), D94.4 (VDD), D95.4 (VDD), D96.4 (VDD), D97.4 (VDD), D98.4 (VDD), J3.1 (Pin_1), SW37.1 (A); no longer J2.2 (Pin_2), JP3.1 (A), JP4.3 (B), R1.1, R2.1, RV1.2, RV2.2
- net GND: now also JP1.3 (B), C1.2, C2.2, D1.2 (VSS), D10.2 (VSS), D11.2 (VSS), D12.2 (VSS), D13.2 (VSS), D14.2 (VSS), D2.2 (VSS), D22.2 (VSS), D23.2 (VSS), D24.2 (VSS), D25.2 (VSS), D26.2 (VSS), D27.2 (VSS), D28.2 (VSS), D29.2 (VSS), D3.2 (VSS), D30.2 (VSS), D31.2 (VSS), D32.2 (VSS), D33.2 (VSS), D34.2 (VSS), D35.2 (VSS), D4.2 (VSS), D43.2 (VSS), D44.2 (VSS), D45.2 (VSS), D46.2 (VSS), D47.2 (VSS), D48.2 (VSS), D49.2 (VSS), D5.2 (VSS), D50.2 (VSS), D51.2 (VSS), D52.2 (VSS), D53.2 (VSS), D54.2 (VSS), D55.2 (VSS), D56.2 (VSS), D6.2 (VSS), D64.2 (VSS), D65.2 (VSS), D66.2 (VSS), D67.2 (VSS), D68.2 (VSS), D69.2 (VSS), D7.2 (VSS), D70.2 (VSS), D71.2 (VSS), D72.2 (VSS), D73.2 (VSS), D74.2 (VSS), D75.2 (VSS), D76.2 (VSS), D77.2 (VSS), D8.2 (VSS), D85.2 (VSS), D86.2 (VSS), D87.2 (VSS), D88.2 (VSS), D89.2 (VSS), D9.2 (VSS), D90.2 (VSS), D91.2 (VSS), D92.2 (VSS), D93.2 (VSS), D94.2 (VSS), D95.2 (VSS), D96.2 (VSS), D97.2 (VSS), D98.2 (VSS), J3.2 (Pin_2), SW35.C, U1.2 (GND); no longer JP3.3 (B)
- net SCL: now also JP3.3 (B); no longer JP1.3 (B)
- net SDA: now also JP4.3 (B); no longer JP2.3 (B)
- net C4: now reaches SW5.1
- net C4: now also SW12.1, SW19.1, SW26.1, SW32.1
- net at SW5.2: now also D19.2 (A)
- net at SW19.2: now also D61.2 (A)
- net C2: now reaches SW30.1
- net C2: now also SW10.1, SW17.1, SW24.1, SW3.1
- net at SW30.2: now also D101.2 (A)
- net at SW26.2: now also D82.2 (A)
- net C0: now reaches SW8.1
- net C0: now also SW1.1, SW15.1, SW22.1, SW28.1
- net at SW8.2: now also D36.2 (A)
- net C5: now reaches SW13.1
- net C5: now also SW20.1, SW27.1, SW33.1, SW6.1
- net at SW13.2: now also D41.2 (A)
- net at SW33.2: now also D104.2 (A)
- net C3: now reaches SW18.1
- net C3: now also SW11.1, SW25.1, SW4.1, SW31.1
- net at SW18.2: now also D60.2 (A)
- net +: now reaches JP5.2 (C)
- net at SW15.2: now also D57.2 (A)
- net at SW27.2: now also D83.2 (A)
- net at SW25.2: now also D81.2 (A)
- net R0: now reaches D15.1 (K)
- net R0: now also D16.1 (K), D17.1 (K), D18.1 (K), D19.1 (K), D20.1 (K), D21.1 (K)
- net at SW11.2: now also D39.2 (A)
- net C6: now reaches SW14.1
- net C6: now also SW21.1, SW34.1, SW7.1, SW35.S1
- net at SW14.2: now also D42.2 (A)
- net at SW24.2: now also D80.2 (A)
- net C1: now reaches SW29.1
- net C1: now also SW16.1, SW2.1, SW23.1, SW9.1
- net at SW29.2: now also D100.2 (A)
- net at SW4.2: now also D18.2 (A)
- net at SW12.2: now also D40.2 (A)
- net at SW3.2: now also D17.2 (A)
- net at SW21.2: now also D63.2 (A)
- net at SW2.2: now also D16.2 (A)
- net at SW6.2: now also D20.2 (A)
- net at SW28.2: now also D99.2 (A)
- net at SW32.2: now also D103.2 (A)
- net at SW10.2: now also D38.2 (A)
- net at SW34.2: now also D105.2 (A)
- net at SW17.2: now also D59.2 (A)
- net at SW7.2: now also D21.2 (A)
- net -: now reaches JP6.2 (C)
- net at SW16.2: now also D58.2 (A)
- net at SW22.2: now also D78.2 (A)
- net at SW9.2: now also D37.2 (A)
- net at SW23.2: now also D79.2 (A)
- net at SW20.2: now also D62.2 (A)
- new net: D49.1 (DOUT), D70.3 (DIN)
- new net: D48.1 (DOUT), D49.3 (DIN)
- new net: C1.1, U1.5 (Vin)
- new net: D89.1 (DOUT), D90.3 (DIN)
- new net: D88.1 (DOUT), D89.3 (DIN)
- new net: D25.3 (DIN), D26.1 (DOUT)
- new net: D26.3 (DIN), D27.1 (DOUT)
- new net: D6.1 (DOUT), D7.3 (DIN)
- new net: D5.1 (DOUT), D6.3 (DIN)
- new net: D27.3 (DIN), D28.1 (DOUT)
- new net: D28.3 (DIN), D7.1 (DOUT)
- new net: D64.3 (DIN), D65.1 (DOUT)
- new net: D65.3 (DIN), D66.1 (DOUT)
- new net: D75.3 (DIN), D76.1 (DOUT)
- new net: D76.3 (DIN), D77.1 (DOUT)
- new net: D71.3 (DIN), D72.1 (DOUT)
- new net: D72.3 (DIN), D73.1 (DOUT)
- new net: D23.3 (DIN), D24.1 (DOUT)
- new net: D24.3 (DIN), D25.1 (DOUT)
- new net: D31.3 (DIN), D32.1 (DOUT)
- new net: D32.3 (DIN), D33.1 (DOUT)
- new net: D47.1 (DOUT), D48.3 (DIN)
- new net: D87.1 (DOUT), D88.3 (DIN)
- new net: D102.2 (A), SW31.2
- new net: D4.1 (DOUT), D5.3 (DIN)
- new net: D22.1 (DOUT), D43.3 (DIN)
- new net: D22.3 (DIN), D23.1 (DOUT)
- new net: D66.3 (DIN), D67.1 (DOUT)
- new net: D90.1 (DOUT), D91.3 (DIN)
- new net: D86.1 (DOUT), D87.3 (DIN)
- new net: D29.1 (DOUT), D50.3 (DIN)
- new net: D29.3 (DIN), D30.1 (DOUT)
- new net: D73.3 (DIN), D74.1 (DOUT)
- new net: D74.3 (DIN), D75.1 (DOUT)
- new net: D67.3 (DIN), D68.1 (DOUT)
- new net: D97.1 (DOUT), D98.3 (DIN)
- new net: D33.3 (DIN), D34.1 (DOUT)
- new net: D3.1 (DOUT), D4.3 (DIN)
- new net: D2.1 (DOUT), D3.3 (DIN)
- new net: D45.1 (DOUT), D46.3 (DIN)
- new net: D44.1 (DOUT), D45.3 (DIN)
- new net: D94.1 (DOUT), D95.3 (DIN)
- new net: D93.1 (DOUT), D94.3 (DIN)
- new net: D96.1 (DOUT), D97.3 (DIN)
- new net: D1.1 (DOUT), D2.3 (DIN)
- new net: D92.1 (DOUT), D93.3 (DIN)
- new net: D71.1 (DOUT), D92.3 (DIN)
- new net: D43.1 (DOUT), D44.3 (DIN)
- new net: D13.1 (DOUT), D14.3 (DIN)
- new net: D12.1 (DOUT), D13.3 (DIN)
- new net: D46.1 (DOUT), D47.3 (DIN)
- new net: D50.1 (DOUT), D51.3 (DIN)
- new net: D10.1 (DOUT), D11.3 (DIN)
- new net: D10.3 (DIN), D9.1 (DOUT)
- new net: D95.1 (DOUT), D96.3 (DIN)
- new net: D85.1 (DOUT), D86.3 (DIN)
- new net: D54.1 (DOUT), D55.3 (DIN)
- new net: D53.1 (DOUT), D54.3 (DIN)
- new net: D55.1 (DOUT), D56.3 (DIN)
- new net: D30.3 (DIN), D31.1 (DOUT)
- new net: D51.1 (DOUT), D52.3 (DIN)
- new net: D8.1 (DOUT), D9.3 (DIN)
- new net: D69.3 (DIN), D70.1 (DOUT)
- new net: D34.3 (DIN), D35.1 (DOUT)
- new net: D68.3 (DIN), D69.1 (DOUT)
- new net: D56.1 (DOUT), D77.3 (DIN)
- new net: D14.1 (DOUT), D35.3 (DIN)
- new net: D64.1 (DOUT), D85.3 (DIN)
- new net: D11.1 (DOUT), D12.3 (DIN)
- new net: D52.1 (DOUT), D53.3 (DIN)
- new net +3.3V: J2.2 (Pin_2), JP2.3 (B), JP3.1 (A), R1.1, R2.1, RV1.2
- new net Bat+: C2.1, U1.4 (Vout)
- new net LED: D1.3 (DIN), D8.3 (DIN)
- new net R1: D36.1 (K), D37.1 (K), D38.1 (K), D39.1 (K), D40.1 (K), D41.1 (K), D42.1 (K)
- new net R2: D57.1 (K), D58.1 (K), D59.1 (K), D60.1 (K), D61.1 (K), D62.1 (K), D63.1 (K)
- new net R3: D78.1 (K), D79.1 (K), D80.1 (K), D81.1 (K), D82.1 (K), D83.1 (K), D84.1 (K)
- new net R4: D100.1 (K), D101.1 (K), D102.1 (K), D103.1 (K), D104.1 (K), D105.1 (K), D99.1 (K)
- new net RE_A: SW35.A
- new net RE_B: SW35.B
- new net RE_S2: D84.2 (A), SW35.S2
- new net VCC: SW37.2 (B)
- no-connect marks 3 -> 6
Other:
- note removed: "dcdc"
- note removed: "qi"
- note removed: "rgbled"
- note removed: "tp4056"
- moved on the sheet: JP5, JP6, SW15, SW16, SW17, SW18, SW19, SW20, SW22, SW23, SW24, SW25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

Commit message: Added Qi charging unit
Parts:
- removed D10, D11, D12, D13, D14, D2, D22, D23, D24, D25, D26, D27, D28, D29, D3, D30, D31, D32, D33, D34, D35, D4, D5, D6, D66, D67, D68, D69, D7, D70, D71, D72, D73, D74, D75, D76, D77, D8, D85, D86, D87, D88, D89, D9, D90, D91, D92, D93, D94, D95, D96, D97, D98: SK6812MINI, LED_SMD:LED_SK6812MINI_PLCC4_3.5x3.5mm_P1.75mm, symbol LED:SK6812MINI
- removed D100, D101, D102, D103, D104, D105, D21, D36, D37, D38, D39, D40, D41, D42, D57, D58, D59, D60, D61, D62, D63, D78, D79, D80, D81, D82, D83, D84, D99: D, Diode_SMD:D_SOD-123, symbol Device:D
- removed J3: Qi Charging unit, symbol Connector:Conn_01x02_Socket
- removed J4: LiPo, symbol Connector:Conn_01x02_Socket
- removed SW14: Command 2, Button_Switch_THT:SW_Tactile_SPST_Angled_PTS645Vx58-2LFS, symbol Switch:SW_Push
- removed SW21: Command 3, Button_Switch_THT:SW_Tactile_SPST_Angled_PTS645Vx58-2LFS, symbol Switch:SW_Push
- removed SW7: Command 1, Button_Switch_THT:SW_Tactile_SPST_Angled_PTS645Vx58-2LFS, symbol Switch:SW_Push
- added BT1: Qi Charging Unit, symbol Device:Battery_Cell
- added BT2: LiPo, symbol Device:Battery_Cell
- added D10, D11, D12, D13, D15, D2, D22, D23, D24, D25, D26, D27, D28, D29, D3, D30, D31, D32, D33, D34, D35, D4, D5, D6, D8, D9: D, Ultramarine-2:SOD-123_reversible, symbol Device:D
- added D37, D38, D39, D40, D41, D42, D57, D58, D59, D60, D61, D62, D63: SK6812MINI, Ultramarine-2:SK6812-mini_reversible, symbol LED:SK6812MINI
- added D66: D, Diode_SMD:D_SOD-123, symbol Device:D
- added F1: Polyfuse_Small, symbol Device:Polyfuse_Small
- added JP7: Power1, Jumper:SolderJumper-3_P2.0mm_Open_TrianglePad1.0x1.5mm, symbol Jumper:Jumper_3_Open
- added JP8: Batt.2, Jumper:SolderJumper-3_P2.0mm_Open_TrianglePad1.0x1.5mm, symbol Jumper:Jumper_3_Open
- added U2, U3: ~, Ultramarine-2:BLE Micro Pro, symbol Ultramarine-2:BLE_micro_Pro
- C1: value C -> 0.33u
- C2: value C -> 2.2u
- D1: renamed from D15; footprint Diode_SMD:D_SOD-123 -> Ultramarine-2:SOD-123_reversible
- D16, D17, D18, D19, D20: footprint Diode_SMD:D_SOD-123 -> Ultramarine-2:SOD-123_reversible
- D36: renamed from D1; footprint LED_SMD:LED_SK6812MINI_PLCC4_3.5x3.5mm_P1.75mm -> Ultramarine-2:SK6812-mini_reversible
- D43, D44, D45, D46, D47, D48, D49, D50, D51, D52, D53, D54, D55, D56, D64, D65: footprint LED_SMD:LED_SK6812MINI_PLCC4_3.5x3.5mm_P1.75mm -> Ultramarine-2:SK6812-mini_reversible
- D67: renamed from D106; value Power -> Power (WH)
- D68: renamed from D107; value Charging -> Charging (OR)
- J1: footprint (none) -> Connector_PinSocket_2.54mm:PinSocket_1x04_P2.54mm_Vertical
- J2: footprint (none) -> Ultramarine-2:MJ-4PP-9
- JP5: value Jumper_3_Open -> Power1; footprint (none) -> Jumper:SolderJumper-3_P2.0mm_Open_TrianglePad1.0x1.5mm
- JP6: value Jumper_3_Open -> Batt.1; footprint (none) -> Jumper:SolderJumper-3_P2.0mm_Open_TrianglePad1.0x1.5mm
- R1, R2: footprint (none) -> Resistor_SMD:R_0603_1608Metric
Connections:
- net +3.3V: now also J2.4 (Pin_4); no longer J2.2 (Pin_2), R1.1, R2.1
- net +5V: now also D43.2 (VSS), D44.2 (VSS), D45.2 (VSS), D46.2 (VSS), D47.2 (VSS), D54.2 (VSS), D55.2 (VSS), D56.2 (VSS), R1.1, R2.1, D37.4 (VDD), D38.4 (VDD), D39.4 (VDD), D40.4 (VDD), D41.4 (VDD), D42.2 (VSS), D57.2 (VSS), D58.2 (VSS), D59.2 (VSS), D60.4 (VDD), D61.4 (VDD), D62.4 (VDD), D63.4 (VDD), D66.1 (K), JP7.1 (A), U2.21 (4.3V), U2.24 (5V), U3.21 (4.3V), U3.24 (5V); no longer D43.4 (VDD), D44.4 (VDD), D45.4 (VDD), D46.4 (VDD), D47.4 (VDD), D54.4 (VDD), D55.4 (VDD), D56.4 (VDD), JP6.1 (A)
- net -: now also JP7.2 (C); no longer JP6.2 (C)
- net Bat+: now also U2.25 (Bat+), U3.25 (Bat+)
- net C0: now also U2.20 (F4), U3.20 (F4)
- net C1: now also U2.19 (F5), U3.19 (F5)
- net C2: now also U2.18 (F6), U3.18 (F6)
- net C3: now also U2.17 (F7), U3.17 (F7)
- net C4: now also U2.16 (B1), U3.16 (B1)
- net C5: now also U2.15 (B3), U3.15 (B3)
- net C6: now also U2.14 (B2), U3.14 (B2)
- net GND: now also D43.4 (VDD), D44.4 (VDD), D45.4 (VDD), D46.4 (VDD), D47.4 (VDD), D54.4 (VDD), D55.4 (VDD), D56.4 (VDD), J2.2 (Pin_2), BT1.2 (-), D37.2 (VSS), D38.2 (VSS), D39.2 (VSS), D40.2 (VSS), D41.2 (VSS), D42.4 (VDD), D57.4 (VDD), D58.4 (VDD), D59.4 (VDD), D60.2 (VSS), D61.2 (VSS), D62.2 (VSS), D63.2 (VSS), JP7.3 (B), U2.0 (GND), U2.23 (GND), U2.3 (GND), U2.4 (GND), U3.0 (GND), U3.23 (GND), U3.3 (GND), U3.4 (GND); no longer D43.2 (VSS), D44.2 (VSS), D45.2 (VSS), D46.2 (VSS), D47.2 (VSS), D54.2 (VSS), D55.2 (VSS), D56.2 (VSS), J2.4 (Pin_4), JP6.3 (B)
- net LED: now also U2.1 (D3), U3.1 (D3)
- net R0: now also D2.1 (K), D3.1 (K), D4.1 (K), D5.1 (K), D6.1 (K), U2.7 (D4), U3.7 (D4); no longer D16.1 (K), D17.1 (K), D18.1 (K), D19.1 (K), D20.1 (K)
- net R1: now also D10.1 (K), D11.1 (K), D12.1 (K), D13.1 (K), D8.1 (K), D9.1 (K), U2.8 (C6), U3.8 (C6)
- net R2: now also D16.1 (K), D17.1 (K), D18.1 (K), D19.1 (K), D20.1 (K), D15.1 (K), U2.9 (D7), U3.9 (D7)
- net R3: now also D22.1 (K), D23.1 (K), D24.1 (K), D25.1 (K), D26.1 (K), D27.1 (K), D28.1 (K), U2.10 (E6), U3.10 (E6)
- net R4: now also D29.1 (K), D30.1 (K), D31.1 (K), D32.1 (K), D33.1 (K), D34.1 (K), D35.1 (K), U2.11 (B4), U3.11 (B4)
- net RE_S2: now also D28.2 (A)
- net SCL: now also U2.6 (D0), U3.6 (D0)
- net SDA: now also U2.5 (D1), U3.5 (D1)
- net data: now also U2.2 (D2), U3.2 (D2)
- net at SW10.2: now also D10.2 (A)
- net at D49.1 (DOUT): now also D50.3 (DIN)
- net at SW2.2: now also D2.2 (A); no longer D16.2 (A)
- net at C1.1, U1.5 (Vin): now also JP6.2 (C), JP8.2 (C)
- net at SW5.2: now also D5.2 (A); no longer D19.2 (A)
- net at SW19.2: now also D19.2 (A)
- net at SW12.2: now also D12.2 (A)
- net at SW34.2: now also D35.2 (A)
- net at SW30.2: now also D31.2 (A)
- net at D64.3 (DIN): now also D63.1 (DOUT); no longer D65.1 (DOUT)
- net at D65.3 (DIN): now also D64.1 (DOUT)
- net at SW26.2: now also D26.2 (A)
- net at SW8.2: now also D8.2 (A)
- net at D18.2 (A): now also SW18.2; no longer SW4.2
- net at SW13.2: now also D13.2 (A)
- net at D48.3 (DIN): now also D42.1 (DOUT); no longer D47.1 (DOUT)
- net at SW31.2: now also D32.2 (A)
- net at SW33.2: now also D34.2 (A)
- net at D43.3 (DIN): now also D44.1 (DOUT)
- net at SW9.2: now also D9.2 (A)
- net at SW15.2: now also D15.2 (A)
- net at SW27.2: now also D27.2 (A)
- net at SW25.2: now also D25.2 (A)
- net at SW28.2: now also D29.2 (A)
- net at SW16.2: now also D16.2 (A)
- net at SW11.2: now also D11.2 (A)
- net at SW24.2: now also D24.2 (A)
- net at D45.1 (DOUT): now also D44.3 (DIN); no longer D46.3 (DIN)
- net at D45.3 (DIN): now also D46.1 (DOUT); no longer D44.1 (DOUT)
- net at SW29.2: now also D30.2 (A)
- net at D17.2 (A): now also SW17.2; no longer SW3.2
- net at D36.1 (DOUT): now also D37.3 (DIN)
- net at D43.1 (DOUT): now also D42.3 (DIN); no longer D44.3 (DIN)
- net at D47.3 (DIN): now also D41.1 (DOUT); no longer D46.1 (DOUT)
- net Charging: now reaches RV2.2
- net Charging: now also BT1.1 (+), D66.2 (A)
- net at D55.3 (DIN): now also D56.1 (DOUT); no longer D54.1 (DOUT)
- net at D54.3 (DIN): now also D55.1 (DOUT); no longer D53.1 (DOUT)
- net at SW20.2: now also D20.2 (A)
- net at SW23.2: now also D23.2 (A)
- net at D56.3 (DIN): now also D57.1 (DOUT); no longer D55.1 (DOUT)
- net at SW6.2: now also D6.2 (A); no longer D20.2 (A)
- net at SW32.2: now also D33.2 (A)
- net at SW22.2: now also D22.2 (A)
- net RESET renamed Reset
- net Reset: now also U2.22 (RST), U3.22 (RST)
- new net: D40.1 (DOUT), D41.3 (DIN)
- new net: D39.1 (DOUT), D40.3 (DIN)
- new net: JP6.1 (A), JP8.3 (B)
- new net: D38.1 (DOUT), D39.3 (DIN)
- new net: D4.2 (A), SW4.2
- new net: D61.1 (DOUT), D62.3 (DIN)
- new net: D60.1 (DOUT), D61.3 (DIN)
- new net: D57.3 (DIN), D58.1 (DOUT)
- new net: D58.3 (DIN), D59.1 (DOUT)
- new net: D37.1 (DOUT), D38.3 (DIN)
- new net: BT2.1 (+), F1.2
- new net: D3.2 (A), SW3.2
- new net: D62.1 (DOUT), D63.3 (DIN)
- new net: D46.3 (DIN), D47.1 (DOUT)
- new net: D53.1 (DOUT), D59.3 (DIN)
- new net: D54.1 (DOUT), D60.3 (DIN)
- no-connect marks 6 -> 9
Other:
- note added: "OLED"
- note added: "Power"
- moved on the sheet: C1, C2, D1, D36, D67, D68, J2, JP5, RV1, RV2, SW1, SW10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
