File: Ultramarine-2.kicad_sch (KiCad schematic)
At the start: 122 parts, among them J1 OLED, J2 TRRS, SW1 SW_Push, SW10 SW_Push, SW11 SW_Push, SW12 SW_Push, SW13 SW_Push, SW15 SW_Push, SW16 SW_Push, SW17 SW_Push, SW18 SW_Push, SW19 SW_Push, SW2 SW_Push, SW20 SW_Push, SW22 SW_Push, SW23 SW_Push, SW24 SW_Push, SW25 SW_Push, SW26 SW_Push, SW27 SW_Push, SW28 SW_Push, SW29 SW_Push, SW3 SW_Push, SW30 SW_Push, SW31 Extra, SW32 SW_Push, SW33 SW_Push, SW34 SW_Push, SW35 RotaryEncoder_Switch, SW36 Reset, SW37 Power Switch, SW4 SW_Push, SW5 SW_Push, SW6 SW_Push, SW8 SW_Push, SW9 SW_Push

Commit message: add PCB patterns
Parts:
- removed D68: Charging (OR), symbol Device:LED
- removed U1: ~, Package_TO_SOT_SMD:SOT-89-5, symbol Ultramarine-2:NJM2884
- removed U4: ~, Ultramarine-2:TP4056, symbol Ultramarine-2:TP4056
- added J3: Flexible LED 3V, Connector_PinSocket_2.54mm:PinSocket_1x01_P2.54mm_Vertical, symbol Connector:Conn_01x01_Socket
- added J4: Flexible LED GND, Connector_PinSocket_2.54mm:PinSocket_1x01_P2.54mm_Vertical, symbol Connector:Conn_01x01_Socket
- added JP9: Flex LED for Power, Jumper:SolderJumper-2_P1.3mm_Open_TrianglePad1.0x1.5mm, symbol Jumper:Jumper_2_Open
- added U3: ~, Ultramarine-2:TP4056, symbol Ultramarine-2:TP4056
- added U4: ~, Package_TO_SOT_SMD:SOT-89-5, symbol Ultramarine-2:NJM2884
- BT1: footprint (none) -> Ultramarine-2:Micro_USB_Charging
- D33: renamed from D36; footprint LED_SMD:LED_SK6812MINI_PLCC4_3.5x3.5mm_P1.75mm -> Ultramarine-2:SK6812-mini_reversible
- D34: renamed from D37; footprint LED_SMD:LED_SK6812MINI_PLCC4_3.5x3.5mm_P1.75mm -> Ultramarine-2:SK6812-mini_reversible
- D35: renamed from D38; footprint LED_SMD:LED_SK6812MINI_PLCC4_3.5x3.5mm_P1.75mm -> Ultramarine-2:SK6812-mini_reversible
- D36: renamed from D39; footprint LED_SMD:LED_SK6812MINI_PLCC4_3.5x3.5mm_P1.75mm -> Ultramarine-2:SK6812-mini_reversible
- D37: renamed from D40; footprint LED_SMD:LED_SK6812MINI_PLCC4_3.5x3.5mm_P1.75mm -> Ultramarine-2:SK6812-mini_reversible
- D38: renamed from D41; footprint LED_SMD:LED_SK6812MINI_PLCC4_3.5x3.5mm_P1.75mm -> Ultramarine-2:SK6812-mini_reversible
- D39: renamed from D42; footprint LED_SMD:LED_SK6812MINI_PLCC4_3.5x3.5mm_P1.75mm -> Ultramarine-2:SK6812-mini_reversible
- D40: renamed from D43; footprint LED_SMD:LED_SK6812MINI_PLCC4_3.5x3.5mm_P1.75mm -> Ultramarine-2:SK6812-mini_reversible
- D41: renamed from D44; footprint LED_SMD:LED_SK6812MINI_PLCC4_3.5x3.5mm_P1.75mm -> Ultramarine-2:SK6812-mini_reversible
- D42: renamed from D45; footprint LED_SMD:LED_SK6812MINI_PLCC4_3.5x3.5mm_P1.75mm -> Ultramarine-2:SK6812-mini_reversible
- D43: renamed from D46; footprint LED_SMD:LED_SK6812MINI_PLCC4_3.5x3.5mm_P1.75mm -> Ultramarine-2:SK6812-mini_reversible
- D44: renamed from D47; footprint LED_SMD:LED_SK6812MINI_PLCC4_3.5x3.5mm_P1.75mm -> Ultramarine-2:SK6812-mini_reversible
- D45: renamed from D48; footprint LED_SMD:LED_SK6812MINI_PLCC4_3.5x3.5mm_P1.75mm -> Ultramarine-2:SK6812-mini_reversible
- D46: renamed from D49; footprint LED_SMD:LED_SK6812MINI_PLCC4_3.5x3.5mm_P1.75mm -> Ultramarine-2:SK6812-mini_reversible
- D47: renamed from D50; footprint LED_SMD:LED_SK6812MINI_PLCC4_3.5x3.5mm_P1.75mm -> Ultramarine-2:SK6812-mini_reversible
- D48: renamed from D51; footprint LED_SMD:LED_SK6812MINI_PLCC4_3.5x3.5mm_P1.75mm -> Ultramarine-2:SK6812-mini_reversible
- D49: renamed from D52; footprint LED_SMD:LED_SK6812MINI_PLCC4_3.5x3.5mm_P1.75mm -> Ultramarine-2:SK6812-mini_reversible
- D50: renamed from D53; footprint LED_SMD:LED_SK6812MINI_PLCC4_3.5x3.5mm_P1.75mm -> Ultramarine-2:SK6812-mini_reversible
- D51: renamed from D54; footprint LED_SMD:LED_SK6812MINI_PLCC4_3.5x3.5mm_P1.75mm -> Ultramarine-2:SK6812-mini_reversible
- D52: renamed from D55; footprint LED_SMD:LED_SK6812MINI_PLCC4_3.5x3.5mm_P1.75mm -> Ultramarine-2:SK6812-mini_reversible
- D53: renamed from D56; footprint LED_SMD:LED_SK6812MINI_PLCC4_3.5x3.5mm_P1.75mm -> Ultramarine-2:SK6812-mini_reversible
- D54: renamed from D57; footprint LED_SMD:LED_SK6812MINI_PLCC4_3.5x3.5mm_P1.75mm -> Ultramarine-2:SK6812-mini_reversible
- D55: renamed from D58; footprint LED_SMD:LED_SK6812MINI_PLCC4_3.5x3.5mm_P1.75mm -> Ultramarine-2:SK6812-mini_reversible
- D56: renamed from D59; footprint LED_SMD:LED_SK6812MINI_PLCC4_3.5x3.5mm_P1.75mm -> Ultramarine-2:SK6812-mini_reversible
- D57: renamed from D60; footprint LED_SMD:LED_SK6812MINI_PLCC4_3.5x3.5mm_P1.75mm -> Ultramarine-2:SK6812-mini_reversible
- D58: renamed from D61; footprint LED_SMD:LED_SK6812MINI_PLCC4_3.5x3.5mm_P1.75mm -> Ultramarine-2:SK6812-mini_reversible
- D59: renamed from D62; footprint LED_SMD:LED_SK6812MINI_PLCC4_3.5x3.5mm_P1.75mm -> Ultramarine-2:SK6812-mini_reversible
- D60: renamed from D63; footprint LED_SMD:LED_SK6812MINI_PLCC4_3.5x3.5mm_P1.75mm -> Ultramarine-2:SK6812-mini_reversible
- D61: renamed from D64; footprint LED_SMD:LED_SK6812MINI_PLCC4_3.5x3.5mm_P1.75mm -> Ultramarine-2:SK6812-mini_reversible
- D62: renamed from D65; footprint LED_SMD:LED_SK6812MINI_PLCC4_3.5x3.5mm_P1.75mm -> Ultramarine-2:SK6812-mini_reversible
- D63: renamed from D66; footprint Diode_SMD:D_SOD-123 -> Ultramarine-2:SOD-123_reversible
- D64: renamed from D67; footprint (none) -> Ultramarine-2:LED1608_reversible
- F1: footprint (none) -> Ultramarine-2:MF-NSMF
- JP1, JP2, JP3, JP4, JP7, JP8: footprint Jumper:SolderJumper-3_P2.0mm_Open_TrianglePad1.0x1.5mm -> Ultramarine-2:Jumper 3pin
- JP5: renamed from JP6; footprint Jumper:SolderJumper-3_P2.0mm_Open_TrianglePad1.0x1.5mm -> Ultramarine-2:Jumper 3pin
- JP6: renamed from JP5; footprint Jumper:SolderJumper-3_P2.0mm_Open_TrianglePad1.0x1.5mm -> Ultramarine-2:Jumper 3pin
- RV1, RV2: footprint (none) -> Ultramarine-2:R_variable
- SW28: renamed from SW31; footprint Button_Switch_THT:SW_Tactile_SPST_Angled_PTS645Vx58-2LFS -> Ultramarine-2:Tactlie_Switch
- SW33: renamed from SW36; footprint Button_Switch_THT:SW_Tactile_SPST_Angled_PTS645Vx58-2LFS -> Ultramarine-2:Tactlie_Switch
- renumbered D11 to D10, D12 to D11, D13 to D12, D15 to D13, D16 to D14, D17 to D15, D18 to D16, D19 to D17, D20 to D18, D22 to D19, D23 to D20, D24 to D21, D25 to D22, D26 to D23, D27 to D24, D28 to D25, D29 to D26, D30 to D27, D31 to D28, D32 to D29, D33 to D30, D34 to D31, D35 to D32, D8 to D7, D9 to D8, D10 to D9, SW11 to SW10, SW12 to SW11, SW13 to SW12, SW15 to SW13, SW16 to SW14, SW17 to SW15, SW18 to SW16, SW19 to SW17, SW20 to SW18, SW22 to SW19, SW23 to SW20, SW24 to SW21, SW25 to SW22, SW26 to SW23, SW27 to SW24, SW28 to SW25, SW29 to SW26, SW30 to SW27, SW32 to SW29, SW33 to SW30, SW34 to SW31, SW35 to SW32, SW37 to SW34, SW8 to SW7, SW9 to SW8, SW10 to SW9, U2 to U1, U3 to U2
Connections:
- net +3.3V: no longer JP2.3 (B), JP3.1 (A), RV1.2
- net +5V: now also JP2.3 (B), JP3.1 (A), JP6.1 (A), JP7.3 (B), RV1.2, JP9.1 (A); no longer JP6.3 (B), JP7.1 (A)
- net Bat+: now also U4.5 (Vout)
- net Charging: now also JP9.2 (B)
- net GND: now also JP5.3 (B), JP6.3 (B), JP7.1 (A), JP8.1 (A), J4.1 (Pin_1), U4.2 (GND); no longer JP6.1 (A), JP7.3 (B)
- net RE_A: now also U1.12 (B5), U2.12 (B5)
- net RE_B: now also U1.13 (B6), U2.13 (B6)
- net at RV2.3: now also J3.1 (Pin_1)
- net at JP6.2 (C): now also U3.1 (+)
- net at JP5.1 (A), JP8.3 (B): now also C1.1, U4.4 (Vin)
- net at F1.1: now also U3.4 (B+)
- net at JP7.2 (C): now also U3.2 (-)
- net at BT2.2 (-): now also U3.5 (B-)
- new net: JP5.2 (C), U3.3 (Out+)
- new net: JP8.2 (C), U3.6 (Out-)
- no-connect marks 9 -> 5
Other:
- moved on the sheet: C1, C2, JP5, JP8
