File: Ultramarine-2_Control_Unit/Ultramarine-2_Control_Unit.kicad_pcb (KiCad board)
At the start: 4 copper layers, 52 x 75 mm, 15 parts, among them J1 TRRS, J2 Generic_connector, J3 Generic_connector, Q1 SSM3J332R, Q2 SSM3J332R, SW1 Slide

Commit message: reversible type
Parts:
- J2, J3: footprint Connector_PinHeader_2.54mm:PinHeader_1x05_P2.54mm_Horizontal -> Ultramarine-2:5pin
- moved J3 8.38 mm to (173.0, 72.7)
- moved J2 8.25 mm to (125.0, 72.7)
Routing:
- net +5V: track 105.4 -> 134.5 mm, vias 3 -> 4
- net Net-(D2-A): track 47.5 -> 25.7 mm
- net /FlexLED: track 45.9 -> 65.8 mm
- net /Bat+: track 67.6 -> 83.9 mm
- net /data: track 67.4 -> 82.3 mm, vias 0 -> 1
- net /Charging: track 31.1 -> 30.6 mm
- net Net-(Q1-G): track 39.7 -> 39.2 mm
- net GND: vias 1 -> 21
Other:
- outline, holes or cut-outs redrawn

Commit message: Changed to 6pin connector
Parts:
- moved BT1 7.07 mm to (149.8, 120.8)
- moved BT2 7.07 mm to (146.0, 78.0)
- moved D1 7.07 mm to (148.5, 106.5)
- moved D2 7.07 mm to (142.8, 122.2)
- moved D3 7.07 mm to (138.5, 113.8)
- moved F1 7.07 mm to (135.3, 113.8)
- moved J1 7.07 mm to (134.0, 50.0)
- moved J2 7.07 mm to (130.0, 77.7)
- moved J3 7.07 mm to (178.0, 77.7)
- moved Q1 7.07 mm to (152.0, 89.9)
- moved Q2 7.07 mm to (152.0, 84.0)
- moved RV1 7.07 mm to (132.5, 102.5)
- moved RV2 7.07 mm to (132.5, 94.8)
- moved SW1 7.07 mm to (135.3, 122.5)
- moved U1 7.07 mm to (146.0, 62.8)
Other:
- board size 52 x 75 mm -> 55 x 75 mm

Commit message: completed version
Parts:
- removed the J2 at (130.0, 77.7)
- removed J3: Generic_connector, Ultramarine-2:5pin
- added G***: LOGO, Ultramarine-2:Chrodream_logo, F.Cu at (165.2, 97.9)
- added G***: LOGO, Ultramarine-2:Chrodream_logo, B.Cu at (164.2, 97.9)
- added J1: Generic_connector, Ultramarine-2:JST_ZH_6, F.Cu at (129.8, 82.0)
- added JP1: OUT+ Jumper, Ultramarine-2:Jumper 3pin, F.Cu at (157.0, 70.4)
- added JP2: IN+ Jumper, Ultramarine-2:Jumper 3pin, F.Cu at (157.0, 53.4)
- added JP3: ~, Ultramarine-2:Jumper 3pin, F.Cu at (157.0, 66.4)
- added JP4: ~, Ultramarine-2:Jumper 3pin, B.Cu at (157.0, 66.4)
- added JP5: ~, Ultramarine-2:Jumper 3pin, F.Cu at (157.0, 57.4)
- added JP6: ~, Ultramarine-2:Jumper 3pin, B.Cu at (157.0, 70.4)
- added JP7: Enable_battery_less_mode, Jumper:SolderJumper-2_P1.3mm_Open_TrianglePad1.0x1.5mm, B.Cu at (139.2, 97.6)
- added U2: ~, Ultramarine-2:TP4056, B.Cu at (146.0, 62.8)
- turned BT1 to 0 degrees
- renumbered BT2 to BT1, BT1 to BT2, D3 to D1, D1 to D2, D2 to D3, J1 to J2
Connections:
- BT1 pad 1: Net-(BT2-+) -> /B+
- BT1 pad 2: Net-(BT2--) -> /B-
- Q1 pad 2: Net-(Q1-G) -> /IN+
- Q1 pad 3: Net-(Q1-S) -> /OUT+
- Q2 pad 1: Net-(Q1-G) -> /IN+
- U1 pad 1: Net-(Q1-G) -> Net-(JP2-C)
- U1 pad 2: GND -> Net-(JP5-C)
- U1 pad 3: Net-(Q1-S) -> Net-(JP6-C)
- U1 pad 4: Net-(BT2-+) -> Net-(JP1-C)
- U1 pad 5: Net-(BT2--) -> Net-(JP3-C)
- U1 pad 6: GND -> Net-(JP4-C)
Routing:
- net /IN+: track 0.00 -> 44.0 mm
- net /data: track 82.3 -> 38.8 mm, vias 1 -> 0
- net /FlexLED: track 65.8 -> 25.3 mm
- net Net-(Q1-G): track 39.2 -> 0.00 mm
- net /OUT+: track 0.00 -> 38.1 mm, vias 0 -> 2
- net /Bat+: track 83.9 -> 45.9 mm
- net /B-: track 0.00 -> 26.9 mm
- net +5V: track 134.6 -> 110.7 mm, vias 4 -> 6
- net Net-(JP4-C): track 0.00 -> 23.8 mm
- net Net-(JP5-C): track 0.00 -> 22.2 mm
- net Net-(JP3-C): track 0.00 -> 20.4 mm
- net /B+: track 0.00 -> 20.1 mm
- net Net-(Q1-S): track 19.6 -> 0.00 mm
- net Net-(JP1-C): track 0.00 -> 9.94 mm
- net Net-(JP6-C): track 0.00 -> 7.76 mm
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Other:
- copper layers 4 -> 2
- board text added: "18650 Li-ion Battery"
