File: Ultramarine-2_Control_Unit/Ultramarine-2_Control_Unit.kicad_sch (KiCad schematic)
At the start: 15 parts, among them J2 Generic_connector, J2 TRRS, J3 Generic_connector, Q1 SSM3J332R, Q2 SSM3J332R, SW33 Slide

Commit message: reversible type
Parts:
- added JP1: Enable_battery_less_mode, symbol Jumper:Jumper_2_Open
- J2, J3: footprint Connector_PinHeader_2.54mm:PinHeader_1x05_P2.54mm_Horizontal -> Ultramarine-2:5pin
Connections:
- net +5V: now also JP1.1 (A)
- net FlexLED: now also JP1.2 (B)
Changed lines of the file:
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@@
+    (stroke (width 0) (type default))
+  )
+  (wire (pts (xy 132.08 254) (xy 142.24 254))
     (stroke (width 0) (type default))
   )
@@
   (label "FlexLED" (at 180.34 215.9 180) (fields_autoplaced)
     (effects (font (size 1.27 1.27)) (justify right bottom))
+  )
+  (label "FlexLED" (at 152.4 254 0) (fields_autoplaced)
+    (effects (font (size 1.27 1.27)) (justify left bottom))
   )
   (label "Bat+" (at 180.34 213.36 180) (fields_autoplaced)
@@
       (effects (font (size 1.27 1.27)) (justify left))
     )
-    (property "Footprint" "Connector_PinHeader_2.54mm:PinHeader_1x05_P2.54mm_Horizontal" (at 215.9 215.9 0)
+    (property "Footprint" "Ultramarine-2:5pin" (at 215.9 215.9 0)
       (effects (font (size 1.27 1.27)) hide)
     )
@@
     )
   )
+  (symbol (lib_id "power:+5V") (at 132.08 254 0) (unit 1)
+    (in_bom yes) (on_board yes) (dnp no) (fields_autoplaced)
+    (property "Reference" "#PWR014" (at 132.08 257.81 0)
+      (effects (font (size 1.27 1.27)) hide)
+    )
+    (property "Value" "+5V" (at 132.08 248.92 0)
+      (effects (font (size 1.27 1.27)))
+    )
+    (property "Footprint" "" (at 132.08 254 0)
+      (effects (font (size 1.27 1.27)) hide)
+    )
+    (property "Datasheet" "" (at 132.08 254 0)
+      (effects (font (size 1.27 1.27)) hide)
+    )
+    (pin "1")
+    (instances
+      (project "Ultramarine-2_Control_Unit"
+        (path "/6d2d31b4-2e7e-4acc-9140-56ecc80c3e53"
+          (reference "#PWR014") (unit 1)
+        )
+      )
+    )
+  )
+  (symbol (lib_id "Jumper:Jumper_2_Open") (at 147.32 254 0) (unit 1)
+    (in_bom yes) (on_board yes) (dnp no) (fields_autoplaced)
+    (property "Reference" "JP1" (at 147.32 247.65 0)
+      (effects (font (size 1.27 1.27)))
+    )
+    (property "Value" "Enable_battery_less_mode" (at 147.32 250.19 0)
+      (effects (font (size 1.27 1.27)))
+    )
+    (property "Footprint" "" (at 147.32 254 0)
+      (effects (font (size 1.27 1.27)) hide)
+    )
+    (property "Datasheet" "~" (at 147.32 254 0)
+      (effects (font (size 1.27 1.27)) hide)
+    )
+    (pin "1")
+    (pin "2")
+    (instances
+      (project "Ultramarine-2_Control_Unit"
+        (path "/6d2d31b4-2e7e-4acc-9140-56ecc80c3e53"
+          (reference "JP1") (unit 1)
+        )
+      )
+    )
+  )
   (symbol (lib_id "Connector:Conn_01x05_Socket") (at 185.42 215.9 0) (unit 1)
     (in_bom yes) (on_board yes) (dnp no) (fields_autoplaced)
@@
       (effects (font (size 1.27 1.27)) (justify left))
     )
-    (property "Footprint" "Connector_PinHeader_2.54mm:PinHeader_1x05_P2.54mm_Horizontal" (at 185.42 215.9 0)
-      (effects (font (size 1.27 1.27)) hide)
-    )
+    (property "Footprint" "Ultramarine-2:5pin" (at 185.42 215.9 0)
+      (effects (font (size 1.27 1.27)) hide)
+    )

Commit message: Changed to 6pin connector
Parts:
- JP1: footprint (none) -> Jumper:SolderJumper-2_P1.3mm_Open_TrianglePad1.0x1.5mm
Changed lines of the file:
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@@
       (effects (font (size 1.27 1.27)))
     )
-    (property "Footprint" "" (at 147.32 254 0)
+    (property "Footprint" "Jumper:SolderJumper-2_P1.3mm_Open_TrianglePad1.0x1.5mm" (at 147.32 254 0)
       (effects (font (size 1.27 1.27)) hide)
     )

Commit message: completed version
Parts:
- removed J2: Generic_connector, Ultramarine-2:5pin, symbol Connector:Conn_01x05_Socket
- added JP1: OUT+ Jumper, Ultramarine-2:Jumper 3pin, symbol Jumper:Jumper_3_Open
- added JP2: IN+ Jumper, Ultramarine-2:Jumper 3pin, symbol Jumper:Jumper_3_Open
- added JP3, JP4, JP5, JP6: ~, Ultramarine-2:Jumper 3pin, symbol Jumper:Jumper_3_Open
- added U2: ~, Ultramarine-2:TP4056, symbol Ultramarine-2:TP4056
- J1: renamed from J3; footprint Ultramarine-2:5pin -> Ultramarine-2:JST_ZH_6; symbol Connector:Conn_01x05_Socket -> Connector:Conn_01x06_Socket
- renumbered JP1 to JP7
Connections:
- net GND: now also JP2.1 (A), JP4.1 (A), JP5.3 (B), JP6.3 (B); no longer U2.2 (-), U2.6 (Out-)
- net IN+: now reaches Q1.2 (G), Q2.1 (D)
- net IN+: now also JP2.3 (B), JP5.1 (A); no longer U2.1 (+)
- net at U2.4 (B+): now also JP1.2 (C), U2.5 (B-); no longer BT2.1 (+)
- net at U2.5 (B-): now also JP3.2 (C), U2.4 (B+); no longer BT2.2 (-)
- net at U2.3 (Out+): now also JP6.2 (C), U2.6 (Out-); no longer Q1.3 (S)
- new net: JP5.2 (C), U2.1 (+), U2.2 (-)
- new net: JP2.2 (C), U2.1 (+), U2.2 (-)
- new net: JP4.2 (C), U2.3 (Out+), U2.6 (Out-)
- new net B+: BT2.1 (+), JP1.3 (B), JP3.1 (A)
- new net B-: BT2.2 (-), JP1.1 (A), JP3.3 (B)
- new net OUT+: JP4.3 (B), JP6.1 (A), Q1.3 (S)
Other:
- moved on the sheet: BT2, D64, F1, Q1, Q2, SW33, U2
